File: CAD/WalkerStalker Shield/WalkerStalkerv20.sch (EAGLE design)
At the start: 25 parts

Commit message: Fixed Temperature sensors
+ Temperature sensors are now called by explicit address, rather than
index, which was not consistent (could not tell if sensor was wall or
air)
+ Unit IDs are not transmitted in data packets for easy identification
+Mounting bracket for TMP006 sensor added (3D file)
Parts:
- removed BH1: BH1750 BOB, SparkFun-Connectors:M04POLAR
- removed DS18B20-1, DS18B20-2: DS18B20, SparkFun-Connectors:M03POLAR
- removed HTU21D: HTU21D BOB, SparkFun-Connectors:M04POLAR
- removed LDR: Mini Photocell, SparkFun-Connectors:M02POLAR
- removed R5: 10K, SparkFun-Resistors:RESISTOR1206
- removed SHT1: SHT15 BOB, SparkFun-Connectors:M04POLAR
- removed TMP1: TMP006 BOB, SparkFun-Connectors:M04POLAR
- removed TSL1: TSL2561 BOB, SparkFun-Connectors:M04POLAR
- added T-AIR, T-WALL: DS18B20, SparkFun-Connectors:M03PTH
- added TMP006: TMP006 BOB, SparkFun-Connectors:M06SIP
- added TSL2561: TSL2561 BOB, SparkFun-Connectors:M04PTH
- MIC: device SparkFun-Connectors:M03POLAR -> SparkFun-Connectors:M03PTH
- R1: value 10K -> 4.7K
- R3, R4: value 15K -> 22K
- RHT1: value RHT03 BOB -> RHT03; device SparkFun-Connectors:M04POLAR -> SparkFun-Connectors:M03PTH
Connections:
- net D4 renamed TF-PWR
- net XBEE-PW renamed XBEE-PWR
- removed net LDR: JP-ANALOG.3, LDR.1, R5.2
- removed net NC: RHT1.2
- removed net SHT15-CL: JP-DIGITAL1.8, SHT1.2
- removed net SHT15-DA: JP-DIGITAL1.7, SHT1.3
- new net A2: JP-ANALOG.3
- new net D6: JP-DIGITAL1.7
- new net D7: JP-DIGITAL1.8
- net +3V3: now also RHT1.3, T-AIR.3, T-WALL.3, TMP006.4, TMP006.6, TSL2561.4; no longer BH1.4, DS18B20-1.3, DS18B20-2.3, HTU21D.4, LDR.2, RHT1.4, SHT1.4, TMP1.4, TSL1.4
- net GND: now also T-AIR.1, T-WALL.1, TMP006.1, TMP006.5, TSL2561.1; no longer BH1.1, DS18B20-1.1, DS18B20-2.1, HTU21D.1, R5.1, SHT1.1, TMP1.1, TSL1.1
- net RHT03: now also R2.1, RHT1.2; no longer R1.1, RHT1.3
- net SCL: now also TMP006.3, TSL2561.3; no longer BH1.3, HTU21D.3, TMP1.3, TSL1.3
- net SDA: now also TMP006.2, TSL2561.2; no longer BH1.2, HTU21D.2, TMP1.2, TSL1.2
- net TEMP_DQ: now also R1.1, T-AIR.2, T-WALL.2; no longer DS18B20-1.2, DS18B20-2.2, R2.1
Other:
- note added: "I²C Addresses DS3231 0x68 TSL2561 0x75 TMP006 0x44"
- note removed: "Connect ADDR pin to +3V3"
- moved on the sheet: R1, R2
